File: RICNU_Plan_v_1_0_SDCard.sch (KiCad schematic (older format))
At the start: 14 parts

Commit message: Added connections to monitor power, changed CANSTB MCU pin, moved LED pins around
Parts:
- D14, D3: value TVS -> 3.3V TVS
Changed lines of the file:
@@
 P 6150 3100
 F 0 "D3" V 6000 3200 50  0000 C CNN
-F 1 "TVS" V 6300 3200 50  0000 C CNN
+F 1 "3.3V TVS" V 6350 3150 50  0000 C CNN
 F 2 "Diodes_SMD:D_SOD-523" H 6150 3100 50  0001 C CNN
 F 3 "" H 6150 3100 50  0001 C CNN
@@
 $EndComp
 $Comp
-L GND #PWR061
+L GND #PWR062
 U 1 1 59FB82E0
 P 3650 5050
-F 0 "#PWR061" H 3650 4800 50  0001 C CNN
+F 0 "#PWR062" H 3650 4800 50  0001 C CNN
 F 1 "GND" H 3650 4900 50  0000 C CNN
 F 2 "" H 3650 5050 50  0001 C CNN
@@
 $EndComp
 $Comp
-L +3V3 #PWR062
+L +3V3 #PWR063
 U 1 1 5A0493ED
 P 3650 2750
-F 0 "#PWR062" H 3650 2600 50  0001 C CNN
+F 0 "#PWR063" H 3650 2600 50  0001 C CNN
 F 1 "+3V3" H 3650 2890 50  0000 C CNN
 F 2 "" H 3650 2750 50  0001 C CNN
@@
 P 7700 4700
 F 0 "D14" V 7550 4800 50  0000 C CNN
-F 1 "TVS" V 7850 4800 50  0000 C CNN
+F 1 "3.3V TVS" V 7850 4800 50  0000 C CNN
 F 2 "Diodes_SMD:D_SOD-523" H 7700 4700 50  0001 C CNN
 F 3 "" H 7700 4700 50  0001 C CNN

Commit message: Various small changes like comment removal
Parts:
- F2: value PTC -> PTC 200 mA
Other:
- note added: "NP"
- note removed: "CPDQC3V3T-HF"
Changed lines of the file:
@@
 P 6400 3100
 F 0 "F2" H 6500 3250 50  0000 C CNN
-F 1 "PTC" H 6550 3150 50  0000 C CNN
+F 1 "PTC 200 mA" H 6750 3150 50  0000 C CNN
 F 2 "Resistors_SMD:R_0603_HandSoldering" H 6450 2900 50  0001 L CNN
 F 3 "" H 6400 3100 50  0001 C CNN
@@
 	0    1    1    0
 $EndComp
-Text Notes 5750 5400 0    60   ~ 0
-CPDQC3V3T-HF
 $Comp
 L R R71
@@
 Connection ~ 7700 4950
 Connection ~ 7950 4950
+Text Notes 6500 3200 0    60   ~ 0
+NP
 $EndSCHEMATC
