File: RICNU_Plan_v_1_0_Manage.sch (KiCad schematic (older format))
At the start: 9 parts, among them J2 MOLEX-PC6

Commit message: Added connections to monitor power, changed CANSTB MCU pin, moved LED pins around
Parts:
- D5: value TVS -> 3.3V TVS
Changed lines of the file:
@@
 P 7150 4400
 F 0 "D5" V 7300 4250 50  0000 C CNN
-F 1 "TVS" H 7150 4300 50  0000 C CNN
+F 1 "3.3V TVS" H 7000 4250 50  0000 C CNN
 F 2 "Diodes_SMD:D_SOD-523" H 7150 4400 50  0001 C CNN
 F 3 "" H 7150 4400 50  0001 C CNN
@@
 CPDQC3V3T-HF
 $Comp
-L +3V3 #PWR063
+L +3V3 #PWR064
 U 1 1 59FB6A2D
 P 4600 3050
-F 0 "#PWR063" H 4600 2900 50  0001 C CNN
+F 0 "#PWR064" H 4600 2900 50  0001 C CNN
 F 1 "+3V3" H 4600 3190 50  0000 C CNN
 F 2 "" H 4600 3050 50  0001 C CNN
@@
 $EndComp
 $Comp
-L GND #PWR064
+L GND #PWR065
 U 1 1 5A050636
 P 4600 5000
-F 0 "#PWR064" H 4600 4750 50  0001 C CNN
+F 0 "#PWR065" H 4600 4750 50  0001 C CNN
 F 1 "GND" H 4600 4850 50  0000 C CNN
 F 2 "" H 4600 5000 50  0001 C CNN

Commit message: Deleting PDFs
Other:
- note removed: "CPDQC3V3T-HF"
- note removed: "TBX0104 on MNG side"
Changed lines of the file:
@@
 	0    1    1    0
 $EndComp
-Text Notes 7300 4450 0    60   ~ 0
-CPDQC3V3T-HF
 $Comp
 L +3V3 #PWR069
@@
 	1    0    0    -1
 $EndComp
-Text Notes 8800 3950 0    60   ~ 0
-TBX0104 on MNG side
 $Comp
 L TPD4E004 TVS3
